File: hardware/LoadCells.sch (KiCad schematic (older format))
At the start: 0 parts

Commit message: Schematic Draft Complete
Parts:
- added C10, C11, C9: 100nF, symbol C
- added J1: GAIN JUMPER, symbol CONN_01X03
- added J2: SPEED JUMPER, symbol CONN_01X03
- added P3: LOAD CELL 1, symbol CONN_01X04
- added P4: LOAD CELL 2, symbol CONN_01X04
- added P5: LOAD CELL 3, symbol CONN_01X04
- added P6: LOAD CELL 4, symbol CONN_01X04
- added U4: ADS1234, symbol ADS1234
Connections:
- new net: C10.2, U4.10 (CAP)
- new net: C10.1, U4.9 (CAP)
- new net +5V: C11.1, P3.1 (P1), P4.1 (P1), P5.1 (P1), P6.1 (P1), U4.20 (REFP), U4.22 (AVDD)
- new net ADC_A0: U4.8 (A0)
- new net ADC_A1: U4.7 (A1)
- new net ADC_DOUT: U4.28 (~DRDY~/DOUT)
- new net ADC_PDWN: U4.26 (~PDWN)
- new net ADC_SCLK: U4.27 (SCLK)
- new net GAIN0: J1.2 (P2), U4.23 (GAIN0)
- new net GND: C11.2, C9.2, J1.3 (P3), J2.3 (P3), P3.4 (P4), P4.4 (P4), P5.4 (P4), P6.4 (P4), U4.19 (REFN), U4.2 (DGND), U4.21 (AGND), U4.3 (CLKIN/XTAL1), U4.5 (DGND), U4.6 (DGND)
- new net LC1N: P3.3 (P3), U4.12 (AINN1)
- new net LC1P: P3.2 (P2), U4.11 (AINP1)
- new net LC2N: P4.3 (P3), U4.17 (AINN2)
- new net LC2P: P4.2 (P2), U4.18 (AINP2)
- new net LC3N: P5.3 (P3), U4.14 (AINN3)
- new net LC3P: P5.2 (P2), U4.13 (AINP3)
- new net LC4N: P6.3 (P3), U4.15 (AINN4)
- new net LC4P: P6.2 (P2), U4.16 (AINP4)
- new net SPEED: J2.2 (P2), U4.25 (SPEED)
- new net VCC: C9.1, J1.1 (P1), J2.1 (P1), U4.1 (DVDD), U4.24 (GAIN1)
- no-connect marks 0 -> 1
Other:
- note added: "GAIN = 64 or 128"
- note added: "JOIN AGND WITH DGND\nUNDER ADS1234"
- note added: "LOAD CELL AMPLIFIER / ADC"
- note added: "LOAD CELL CONNECTORS\n"
- note added: "SPEED = 10SPS or 80SPS"

Commit message: PCB mostly routed
Parts:
- C10, C11, C9: footprint (none) -> Resistors_SMD:R_0805_HandSoldering
- J1, J2: footprint (none) -> Pin_Headers:Pin_Header_Straight_1x03
- P3, P4, P5, P6: footprint (none) -> autokiln:ostoq047151
- U4: footprint (none) -> Housings_SSOP:TSSOP-28_4.4x9.7mm_Pitch0.65mm
Changed lines of the file:
@@
 encoding utf-8
 Sheet 3 6
-Title ""
-Date ""
-Rev ""
-Comp ""
+Title "Wood Drying Kiln Controller \"AutoKiln\""
+Date "Sat 21 Mar 2015"
+Rev "A1"
+Comp "Chris Merck"
 Comment1 ""
 Comment2 ""
@@
 F 0 "U4" H 5450 5250 60  0000 C CNN
 F 1 "ADS1234" H 5450 5150 60  0000 C CNN
-F 2 "" H 5450 5250 60  0000 C CNN
+F 2 "Housings_SSOP:TSSOP-28_4.4x9.7mm_Pitch0.65mm" H 5450 5250 60  0001 C CNN
 F 3 "" H 5450 5250 60  0000 C CNN
 	1    5450 3750
@@
 	7750 3550 7750 3800
 $Comp
-L +5V #PWR33
+L +5V #PWR022
 U 1 1 550D6C2D
 P 7750 3550
-F 0 "#PWR33" H 7750 3400 60  0001 C CNN
+F 0 "#PWR022" H 7750 3400 60  0001 C CNN
 F 1 "+5V" H 7750 3690 60  0000 C CNN
 F 2 "" H 7750 3550 60  0000 C CNN
@@
 F 0 "C11" H 7775 4050 50  0000 L CNN
 F 1 "100nF" H 7775 3850 50  0000 L CNN
-F 2 "" H 7788 3800 30  0000 C CNN
+F 2 "Resistors_SMD:R_0805_HandSoldering" H 7788 3800 30  0001 C CNN
 F 3 "" H 7750 3950 60  0000 C CNN
 	1    7750 3950
@@
 	7750 4100 7750 4200
 $Comp
-L GND #PWR34
+L GND #PWR023
 U 1 1 550D6C66
 P 7750 4200
-F 0 "#PWR34" H 7750 3950 60  0001 C CNN
+F 0 "#PWR023" H 7750 3950 60  0001 C CNN
 F 1 "GND" H 7750 4050 60  0000 C CNN
 F 2 "" H 7750 4200 60  0000 C CNN
@@
 F 0 "C10" H 3925 4350 50  0000 L CNN
 F 1 "100nF" H 3925 4150 50  0000 L CNN
-F 2 "" H 3938 4100 30  0000 C CNN
+F 2 "Resistors_SMD:R_0805_HandSoldering" H 3938 4100 30  0001 C CNN
 F 3 "" H 3900 4250 60  0000 C CNN
 	1    3900 4250
@@
 	4100 4350 4700 4350
 $Comp
-L GND #PWR32
+L GND #PWR024
 U 1 1 550D6DA4
 P 6500 3950
-F 0 "#PWR32" H 6500 3700 60  0001 C CNN
+F 0 "#PWR024" H 6500 3700 60  0001 C CNN
 F 1 "GND" V 6500 3750 60  0000 C CNN
 F 2 "" H 6500 3950 60  0000 C CNN
@@
 	4400 2550 4400 2400
 $Comp
-L VCC #PWR27
+L VCC #PWR025
 U 1 1 550D6E23
 P 4400 2400
-F 0 "#PWR27" H 4400 2250 60  0001 C CNN
+F 0 "#PWR025" H 4400 2250 60  0001 C CNN
 F 1 "VCC" H 4400 2550 60  0000 C CNN
 F 2 "" H 4400 2400 60  0000 C CNN
@@
 	4400 2750 4700 2750
 $Comp
-L GND #PWR28
+L GND #PWR026
 U 1 1 550D6E4F
 P 4400 2750
-F 0 "#PWR28" H 4400 2500 60  0001 C CNN
+F 0 "#PWR026" H 4400 2500 60  0001 C CNN
 F 1 "GND" V 4400 2550 60  0000 C CNN
 F 2 "" H 4400 2750 60  0000 C CNN
@@
 	4700 3350 4400 3350
 $Comp
-L GND #PWR29
+L GND #PWR027
 U 1 1 550D6EE9
 P 4400 3350
-F 0 "#PWR29" H 4400 3100 60  0001 C CNN
+F 0 "#PWR027" H 4400 3100 60  0001 C CNN
 F 1 "GND" V 4400 3150 60  0000 C CNN
 F 2 "" H 4400 3350 60  0000 C CNN
@@
 	4700 3550 4400 3550
 $Comp
-L GND #PWR30
+L GND #PWR028
 U 1 1 550D6EF6
 P 4400 3550
-F 0 "#PWR30" H 4400 3300 60  0001 C CNN
+F 0 "#PWR028" H 4400 3300 60  0001 C CNN
 F 1 "GND" V 4400 3350 60  0000 C CNN
 F 2 "" H 4400 3550 60  0000 C CNN
@@
 	6200 3550 6600 3550
 $Comp
-L VCC #PWR31
+L VCC #PWR029
 U 1 1 550D723C
 P 6500 3350
-F 0 "#PWR31" H 6500 3200 60  0001 C CNN
+F 0 "#PWR029" H 6500 3200 60  0001 C CNN
 F 1 "VCC" V 6500 3550 60  0000 C CNN
 F 2 "" H 6500 3350 60  0000 C CNN
@@
 F 0 "P3" H 1600 2600 50  0000 C CNN
 F 1 "LOAD CELL 1" H 1950 2350 50  0000 C CNN
-F 2 "" H 1600 2350 60  0000 C CNN
+F 2 "autokiln:ostoq047151" H 1600 2350 60  0001 C CNN
 F 3 "" H 1600 2350 60  0000 C CNN
 	1    1600 2350
@@
 	1800 2400 2200 2400
 $Comp
-L GND #PWR20
+L GND #PWR030
 U 1 1 550D7644
 P 2000 2600
-F 0 "#PWR20" H 2000 2350 60  0001 C CNN
+F 0 "#PWR030" H 2000 2350 60  0001 C CNN
 F 1 "GND" H 2000 2450 60  0000 C CNN
 F 2 "" H 2000 2600 60  0000 C CNN
@@
 	2000 2100 2000 2200
 $Comp
-L +5V #PWR19
+L +5V #PWR031
 U 1 1 550D76CA
 P 2000 2100
-F 0 "#PWR19" H 2000 1950 60  0001 C CNN
+F 0 "#PWR031" H 2000 1950 60  0001 C CNN
 F 1 "+5V" H 2000 2240 60  0000 C CNN
 F 2 "" H 2000 2100 60  0000 C CNN
@@
 F 0 "P4" H 1600 3650 50  0000 C CNN
 F 1 "LOAD CELL 2" H 1950 3400 50  0000 C CNN
-F 2 "" H 1600 3400 60  0000 C CNN
+F 2 "autokiln:ostoq047151" H 1600 3400 60  0001 C CNN
 F 3 "" H 1600 3400 60  0000 C CNN
 	1    1600 3400
@@
 	1800 3450 2200 3450
 $Comp
-L GND #PWR22
+L GND #PWR032
 U 1 1 550D7782
 P 2000 3650
-F 0 "#PWR22" H 2000 3400 60  0001 C CNN
+F 0 "#PWR032" H 2000 3400 60  0001 C CNN
 F 1 "GND" H 2000 3500 60  0000 C CNN
 F 2 "" H 2000 3650 60  0000 C CNN
@@
 	2000 3150 2000 3250
 $Comp
-L +5V #PWR21
+L +5V #PWR033
 U 1 1 550D778C
 P 2000 3150
-F 0 "#PWR21" H 2000 3000 60  0001 C CNN
+F 0 "#PWR033" H 2000 3000 60  0001 C CNN
 F 1 "+5V" H 2000 3290 60  0000 C CNN
 F 2 "" H 2000 3150 60  0000 C CNN
@@
 F 0 "P5" H 1600 4700 50  0000 C CNN
 F 1 "LOAD CELL 3" H 1950 4450 50  0000 C CNN
-F 2 "" H 1600 4450 60  0000 C CNN
+F 2 "autokiln:ostoq047151" H 1600 4450 60  0001 C CNN
 F 3 "" H 1600 4450 60  0000 C CNN
 	1    1600 4450
@@
 	1800 4500 2200 4500
 $Comp
-L GND #PWR24
+L GND #PWR034
 U 1 1 550D78B1
 P 2000 4700
-F 0 "#PWR24" H 2000 4450 60  0001 C CNN
+F 0 "#PWR034" H 2000 4450 60  0001 C CNN
 F 1 "GND" H 2000 4550 60  0000 C CNN
 F 2 "" H 2000 4700 60  0000 C CNN
@@
 	2000 4200 2000 4300
 $Comp
-L +5V #PWR23
+L +5V #PWR035
 U 1 1 550D78BB
 P 2000 4200
-F 0 "#PWR23" H 2000 4050 60  0001 C CNN
+F 0 "#PWR035" H 2000 4050 60  0001 C CNN
 F 1 "+5V" H 2000 4340 60  0000 C CNN
 F 2 "" H 2000 4200 60  0000 C CNN
@@
 F 0 "P6" H 1600 5750 50  0000 C CNN
 F 1 "LOAD CELL 4" H 1950 5500 50  0000 C CNN
-F 2 "" H 1600 5500 60  0000 C CNN
+F 2 "autokiln:ostoq047151" H 1600 5500 60  0001 C CNN
 F 3 "" H 1600 5500 60  0000 C CNN
 	1    1600 5500
@@
 	1800 5550 2200 5550
 $Comp
-L GND #PWR26
+L GND #PWR036
 U 1 1 550D78CB
 P 2000 5750
-F 0 "#PWR26" H 2000 5500 60  0001 C CNN
+F 0 "#PWR036" H 2000 5500 60  0001 C CNN
 F 1 "GND" H 2000 5600 60  0000 C CNN
 F 2 "" H 2000 5750 60  0000 C CNN
@@
 	2000 5250 2000 5350
 $Comp
-L +5V #PWR25
+L +5V #PWR037
 U 1 1 550D78D5
 P 2000 5250
-F 0 "#PWR25" H 2000 5100 60  0001 C CNN
+F 0 "#PWR037" H 2000 5100 60  0001 C CNN
 F 1 "+5V" H 2000 5390 60  0000 C CNN
 F 2 "" H 2000 5250 60  0000 C CNN
@@
 F 0 "J1" H 10100 3500 50  0000 C CNN
 F 1 "GAIN JUMPER" H 10400 3300 50  0000 C CNN
-F 2 "" H 10100 3300 60  0000 C CNN
+F 2 "Pin_Headers:Pin_Header_Straight_1x03" H 10100 3300 60  0001 C CNN
 F 3 "" H 10100 3300 60  0000 C CNN
 	1    10100 3300
@@
 	9800 3400 9800 3450
 $Comp
-L VCC #PWR35
+L VCC #PWR038
 U 1 1 550D84D9
 P 9800 3100
-F 0 "#PWR35" H 9800 2950 60  0001 C CNN
+F 0 "#PWR038" H 9800 2950 60  0001 C CNN
 F 1 "VCC" H 9800 3250 60  0000 C CNN
 F 2 "" H 9800 3100 60  0000 C CNN
@@
 $EndComp
 $Comp
-L GND #PWR36
+L GND #PWR039
 U 1 1 550D8533
 P 9800 3450
-F 0 "#PWR36" H 9800 3200 60  0001 C CNN
+F 0 "#PWR039" H 9800 3200 60  0001 C CNN
 F 1 "GND" H 9800 3300 60  0000 C CNN
 F 2 "" H 9800 3450 60  0000 C CNN
@@
 F 0 "J2" H 10100 4950 50  0000 C CNN
 F 1 "SPEED JUMPER" H 10500 4750 50  0000 C CNN
-F 2 "" H 10100 4750 60  0000 C CNN
+F 2 "Pin_Headers:Pin_Header_Straight_1x03" H 10100 4750 60  0001 C CNN
 F 3 "" H 10100 4750 60  0000 C CNN
 	1    10100 4750
@@
 	9800 4850 9800 4900
 $Comp
-L VCC #PWR37
+L VCC #PWR040
 U 1 1 550D878F
 P 9800 4550
-F 0 "#PWR37" H 9800 4400 60  0001 C CNN
+F 0 "#PWR040" H 9800 4400 60  0001 C CNN
 F 1 "VCC" H 9800 4700 60  0000 C CNN
 F 2 "" H 9800 4550 60  0000 C CNN
@@
 $EndComp
 $Comp
-L GND #PWR38
+L GND #PWR041
 U 1 1 550D8795
 P 9800 4900
-F 0 "#PWR38" H 9800 4650 60  0001 C CNN
+F 0 "#PWR041" H 9800 4650 60  0001 C CNN
 F 1 "GND" H 9800 4750 60  0000 C CNN
 F 2 "" H 9800 4900 60  0000 C CNN
@@
 F 0 "C9" H 3775 2800 50  0000 L CNN
 F 1 "100nF" H 3775 2600 50  0000 L CNN
-F 2 "" H 3788 2550 30  0000 C CNN
+F 2 "Resistors_SMD:R_0805_HandSoldering" H 3788 2550 30  0001 C CNN
 F 3 "" H 3750 2700 60  0000 C CNN
 	1    3750 2700
