File: hardware/Power.sch (KiCad schematic (older format))
At the start: 9 parts

Commit message: Schematic Draft Complete
Parts:
- added C14: 4u7, symbol C
- added C15: 100uF, symbol C
- added U6: 7805, symbol 7805
- C12: renamed from C?; value 2u2 -> 4u7
- gave numbers to parts that had none: 8
Connections:
- net +12V: now also C14.1, U6.VI; no longer C17.1, U7.8 (VIN)
- net GND: now also C14.2, C15.2, U6.GND
- new net +5V: C15.1, C17.1, U6.VO, U7.8 (VIN)
Other:
- note added: "5V SUPPLY"
- moved on the sheet: C12, C13, C16, C17, D6, P15, SW5, U7, U8

Commit message: PCB mostly routed
Parts:
- removed U6: 7805, symbol 7805
- added U6: L7805, autokiln:TO-220_SG, symbol L7805
- C12, C14: footprint (none) -> Resistors_SMD:R_0805_HandSoldering
- C13, C15, C16, C17: footprint (none) -> autokiln:KEMET_100uF_25V
- D6: footprint (none) -> Diodes_ThroughHole:Diode_LED_5mm_round_vertical
- P15: footprint (none) -> autokiln:CUI_PJ-002AH_DC_PWR_JACK; symbol CONN_01X02 -> CONN_01X03
- SW5: footprint (none) -> autokiln:ESwitch-100SP1T1B4M2QE
- U7: footprint (none) -> Power_Integrations:SO-8
- U8: footprint TO-220-4 -> autokiln:TO-220F-4L
Connections:
- wire segments 39 -> 40
Other:
- note added: "barrel"
Changed lines of the file:
@@
 encoding utf-8
 Sheet 6 6
-Title ""
-Date ""
-Rev ""
-Comp ""
+Title "Wood Drying Kiln Controller \"AutoKiln\""
+Date "Sat 21 Mar 2015"
+Rev "A1"
+Comp "Chris Merck"
 Comment1 ""
 Comment2 ""
@@
 $EndDescr
 $Comp
-L CONN_01X02 P15
+L CONN_01X03 P15
 U 1 1 55065FE1
-P 3400 1350
-F 0 "P15" H 3400 1500 50  0000 C CNN
-F 1 "VIN" H 3550 1400 50  0000 C CNN
-F 2 "" H 3400 1350 60  0000 C CNN
-F 3 "" H 3400 1350 60  0000 C CNN
-	1    3400 1350
+P 3400 1400
+F 0 "P15" H 3400 1600 50  0000 C CNN
+F 1 "VIN" H 3550 1500 50  0000 C CNN
+F 2 "autokiln:CUI_PJ-002AH_DC_PWR_JACK" H 3400 1400 60  0001 C CNN
+F 3 "" H 3400 1400 60  0000 C CNN
+	1    3400 1400
 	-1   0    0    -1
 $EndComp
@@
 	3600 1400 3700 1400
 Wire Wire Line
-	3700 1400 3700 1450
-$Comp
-L GND #PWR53
+	3700 1400 3700 1650
+$Comp
+L GND #PWR056
 U 1 1 550660E3
-P 3700 1450
-F 0 "#PWR53" H 3700 1200 60  0001 C CNN
-F 1 "GND" H 3700 1300 60  0000 C CNN
-F 2 "" H 3700 1450 60  0000 C CNN
-F 3 "" H 3700 1450 60  0000 C CNN
-	1    3700 1450
+P 3700 1650
+F 0 "#PWR056" H 3700 1400 60  0001 C CNN
+F 1 "GND" H 3700 1500 60  0000 C CNN
+F 2 "" H 3700 1650 60  0000 C CNN
+F 3 "" H 3700 1650 60  0000 C CNN
+	1    3700 1650
 	1    0    0    -1
 $EndComp
@@
 F 0 "U8" H 4800 1550 40  0000 C CNN
 F 1 "KA278R12C" H 4950 1550 40  0000 L CNN
-F 2 "TO-220-4" H 5000 1450 30  0000 C CIN
+F 2 "autokiln:TO-220F-4L" H 5000 1700 30  0001 C CIN
 F 3 "" H 5000 1350 60  0000 C CNN
 	1    5000 1350
@@
 	5800 1200 5800 1450
 $Comp
-L +12V #PWR61
+L +12V #PWR057
 U 1 1 55066344
 P 5800 1200
-F 0 "#PWR61" H 5800 1050 60  0001 C CNN
+F 0 "#PWR057" H 5800 1050 60  0001 C CNN
 F 1 "+12V" H 5800 1340 60  0000 C CNN
 F 2 "" H 5800 1200 60  0000 C CNN
@@
 	5000 1650 5000 2100
 $Comp
-L GND #PWR58
+L GND #PWR058
 U 1 1 5506636C
 P 5000 2100
-F 0 "#PWR58" H 5000 1850 60  0001 C CNN
+F 0 "#PWR058" H 5000 1850 60  0001 C CNN
 F 1 "GND" H 5000 1950 60  0000 C CNN
 F 2 "" H 5000 2100 60  0000 C CNN
@@
 F 0 "SW5" H 3950 2400 50  0000 C CNN
 F 1 "PWR SWITCH" H 3950 2200 50  0000 C CNN
-F 2 "" H 3950 2300 60  0000 C CNN
+F 2 "autokiln:ESwitch-100SP1T1B4M2QE" H 3950 2300 60  0001 C CNN
 F 3 "" H 3950 2300 60  0000 C CNN
 	1    3950 2300
@@
 F 0 "C13" H 4075 1750 50  0000 L CNN
 F 1 "100uF" H 4075 1550 50  0000 L CNN
-F 2 "" H 4088 1500 30  0000 C CNN
+F 2 "autokiln:KEMET_100uF_25V" H 4088 1500 30  0001 C CNN
 F 3 "" H 4050 1650 60  0000 C CNN
 	1    4050 1650
@@
 F 0 "C16" H 5825 1700 50  0000 L CNN
 F 1 "100uF" H 5825 1500 50  0000 L CNN
-F 2 "" H 5838 1450 30  0000 C CNN
+F 2 "autokiln:KEMET_100uF_25V" H 5838 1450 30  0001 C CNN
 F 3 "" H 5800 1600 60  0000 C CNN
 	1    5800 1600
@@
 	4900 7300 4900 7400
 $Comp
-L GND #PWR57
+L GND #PWR059
 U 1 1 55066AE6
 P 4900 7400
-F 0 "#PWR57" H 4900 7150 60  0001 C CNN
+F 0 "#PWR059" H 4900 7150 60  0001 C CNN
 F 1 "GND" H 4900 7250 60  0000 C CNN
 F 2 "" H 4900 7400 60  0000 C CNN
@@
 	3700 6200 3700 6700
 $Comp
-L VCC #PWR54
+L VCC #PWR060
 U 1 1 55066B45
 P 3700 6200
-F 0 "#PWR54" H 3700 6050 60  0001 C CNN
+F 0 "#PWR060" H 3700 6050 60  0001 C CNN
 F 1 "VCC" H 3700 6350 60  0000 C CNN
 F 2 "" H 3700 6200 60  0000 C CNN
@@
 	5650 6100 5650 6350
 $Comp
-L +12V #PWR55
+L +12V #PWR061
 U 1 1 55066BBF
 P 4200 3800
-F 0 "#PWR55" H 4200 3650 60  0001 C CNN
+F 0 "#PWR061" H 4200 3650 60  0001 C CNN
 F 1 "+12V" H 4200 3940 60  0000 C CNN
 F 2 "" H 4200 3800 60  0000 C CNN
@@
 F 0 "U7" H 4900 6850 60  0000 C CNN
 F 1 "L4931" H 4900 6750 60  0000 C CNN
-F 2 "" H 4900 6850 60  0000 C CNN
+F 2 "Power_Integrations:SO-8" H 4900 6850 60  0001 C CNN
 F 3 "" H 4900 6850 60  0000 C CNN
 	1    4900 6450
@@
 F 0 "C17" H 6125 6900 50  0000 L CNN
 F 1 "100uF" H 6125 6700 50  0000 L CNN
-F 2 "" H 6138 6650 30  0000 C CNN
+F 2 "autokiln:KEMET_100uF_25V" H 6138 6650 30  0001 C CNN
 F 3 "" H 6100 6800 60  0000 C CNN
 	1    6100 6800
@@
 F 0 "C12" H 3725 6950 50  0000 L CNN
 F 1 "4u7" H 3725 6750 50  0000 L CNN
-F 2 "" H 3738 6700 30  0000 C CNN
+F 2 "Resistors_SMD:R_0805_HandSoldering" H 3738 6700 30  0001 C CNN
 F 3 "" H 3700 6850 60  0000 C CNN
 	1    3700 6850
@@
 F 0 "D6" V 6200 1450 50  0000 C CNN
 F 1 "12V LED" V 6550 1350 50  0000 C CNN
-F 2 "" H 6350 1600 60  0000 C CNN
+F 2 "Diodes_ThroughHole:Diode_LED_5mm_round_vertical" H 6350 1600 60  0001 C CNN
 F 3 "" H 6350 1600 60  0000 C CNN
 	1    6350 1600
@@
 Connection ~ 5800 2000
 $Comp
-L +5V #PWR60
+L +5V #PWR062
 U 1 1 55085518
 P 5650 6100
-F 0 "#PWR60" H 5650 5950 60  0001 C CNN
+F 0 "#PWR062" H 5650 5950 60  0001 C CNN
 F 1 "+5V" H 5650 6240 60  0000 C CNN
 F 2 "" H 5650 6100 60  0000 C CNN
 F 3 "" H 5650 6100 60  0000 C CNN
 	1    5650 6100
-	1    0    0    -1
-$EndComp
-$Comp
-L 7805 U6
-U 1 1 55085A35
-P 4900 4100
-F 0 "U6" H 4900 4450 60  0000 C CNN
-F 1 "7805" H 4900 4300 60  0000 C CNN
-F 2 "" H 4900 4100 60  0000 C CNN
-F 3 "" H 4900 4100 60  0000 C CNN
-	1    4900 4100
 	1    0    0    -1
 $EndComp
@@
 F 0 "C15" H 5575 4500 50  0000 L CNN
 F 1 "100uF" H 5575 4300 50  0000 L CNN
-F 2 "" H 5588 4250 30  0000 C CNN
+F 2 "autokiln:KEMET_100uF_25V" H 5588 4250 30  0001 C CNN
 F 3 "" H 5550 4400 60  0000 C CNN
 	1    5550 4400
@@
 F 0 "C14" H 4225 4500 50  0000 L CNN
 F 1 "4u7" H 4225 4300 50  0000 L CNN
-F 2 "" H 4238 4250 30  0000 C CNN
+F 2 "Resistors_SMD:R_0805_HandSoldering" H 4238 4250 30  0001 C CNN
 F 3 "" H 4200 4400 60  0000 C CNN
 	1    4200 4400
@@
 $EndComp
 $Comp
-L GND #PWR56
+L GND #PWR063
 U 1 1 55085DBB
 P 4900 4850
-F 0 "#PWR56" H 4900 4600 60  0001 C CNN
+F 0 "#PWR063" H 4900 4600 60  0001 C CNN
 F 1 "GND" H 4900 4700 60  0000 C CNN
 F 2 "" H 4900 4850 60  0000 C CNN
@@
 $EndComp
 $Comp
-L +5V #PWR59
+L +5V #PWR064
 U 1 1 55085DDE
 P 5550 3800
-F 0 "#PWR59" H 5550 3650 60  0001 C CNN
+F 0 "#PWR064" H 5550 3650 60  0001 C CNN
 F 1 "+5V" H 5550 3940 60  0000 C CNN
 F 2 "" H 5550 3800 60  0000 C CNN
@@
 	4200 3800 4200 4250
 Wire Wire Line
-	4500 4050 4200 4050
+	4200 4050 4550 4050
 Connection ~ 4200 4050
-Wire Wire Line
-	4900 4350 4900 4850
 Wire Wire Line
 	4200 4550 4200 4700
@@
 	5550 3800 5550 4250
 Wire Wire Line
-	5300 4050 5550 4050
+	5250 4050 5550 4050
 Connection ~ 5550 4050
 Text Notes 4700 3500 0    60   ~ 0
 5V SUPPLY
+Text Notes 3300 1700 0    60   ~ 0
+barrel
+Wire Wire Line
+	3600 1500 3700 1500
+Connection ~ 3700 1500
+$Comp
+L L7805 U6
+U 1 1 550F0F34
+P 4900 4200
+F 0 "U6" H 4900 4600 60  0000 C CNN
+F 1 "L7805" H 4900 4500 60  0000 C CNN
+F 2 "autokiln:TO-220_SG" H 4900 4500 60  0001 C CNN
+F 3 "" H 4900 4500 60  0000 C CNN
+	1    4900 4200
+	1    0    0    -1
+$EndComp
+Wire Wire Line
+	4900 4850 4900 4450
 $EndSCHEMATC
