File: hardware/Sensors.sch (KiCad schematic (older format))
At the start: 5 parts

Commit message: Schematic Draft Complete
Parts:
- added J3: HUMID PWR, symbol CONN_01X03
- added P14: HUMID2, symbol CONN_01X03
- added R4: 1k, symbol R
- P13: renamed from P?; value HUMID -> HUMID1
- gave numbers to parts that had none: 4
Connections:
- net labels added: +5V, HUMID_DATA1, HUMID_DATA2, HUMID_PWR
- net labels removed: HUMID_DATA
- wire segments 27 -> 36
Other:
- moved on the sheet: P12, P13, R2, R3, R5

Commit message: PCB mostly routed
Parts:
- J3: footprint (none) -> Pin_Headers:Pin_Header_Straight_1x03
- P12: footprint (none) -> autokiln:ostoq047151
- P13, P14: footprint (none) -> autokiln:OSTOQ037151
- R2, R3, R4, R5: footprint (none) -> Resistors_SMD:R_0805_HandSoldering
Changed lines of the file:
@@
 encoding utf-8
 Sheet 5 6
-Title ""
-Date ""
-Rev ""
-Comp ""
+Title "Wood Drying Kiln Controller \"AutoKiln\""
+Date "Sat 21 Mar 2015"
+Rev "A1"
+Comp "Chris Merck"
 Comment1 ""
 Comment2 ""
@@
 F 0 "P13" H 5650 2200 50  0000 C CNN
 F 1 "HUMID1" H 5850 2050 50  0000 C CNN
-F 2 "" H 5650 2000 60  0000 C CNN
+F 2 "autokiln:OSTOQ037151" H 5650 2000 60  0001 C CNN
 F 3 "" H 5650 2000 60  0000 C CNN
 	1    5650 2000
@@
 	5950 2100 5950 2200
 $Comp
-L GND #PWR49
+L GND #PWR050
 U 1 1 5506578A
 P 5950 2200
-F 0 "#PWR49" H 5950 1950 60  0001 C CNN
+F 0 "#PWR050" H 5950 1950 60  0001 C CNN
 F 1 "GND" H 5950 2050 60  0000 C CNN
 F 2 "" H 5950 2200 60  0000 C CNN
@@
 F 0 "R3" V 6280 1900 50  0000 C CNN
 F 1 "1k" V 6200 1900 50  0000 C CNN
-F 2 "" V 6130 1900 30  0000 C CNN
+F 2 "Resistors_SMD:R_0805_HandSoldering" V 6130 1900 30  0001 C CNN
 F 3 "" H 6200 1900 30  0000 C CNN
 	1    6200 1900
@@
 F 0 "P12" H 5500 5350 50  0000 C CNN
 F 1 "BAROM" H 5700 5100 50  0000 C CNN
-F 2 "" H 5500 5100 60  0000 C CNN
+F 2 "autokiln:ostoq047151" H 5500 5100 60  0001 C CNN
 F 3 "" H 5500 5100 60  0000 C CNN
 	1    5500 5100
@@
 	5850 4750 5850 4950
 $Comp
-L VCC #PWR47
+L VCC #PWR051
 U 1 1 55065B60
 P 5850 4750
-F 0 "#PWR47" H 5850 4600 60  0001 C CNN
+F 0 "#PWR051" H 5850 4600 60  0001 C CNN
 F 1 "VCC" H 5850 4900 60  0000 C CNN
 F 2 "" H 5850 4750 60  0000 C CNN
@@
 	5850 5250 5850 5350
 $Comp
-L GND #PWR48
+L GND #PWR052
 U 1 1 55065BB3
 P 5850 5350
-F 0 "#PWR48" H 5850 5100 60  0001 C CNN
+F 0 "#PWR052" H 5850 5100 60  0001 C CNN
 F 1 "GND" H 5850 5200 60  0000 C CNN
 F 2 "" H 5850 5350 60  0000 C CNN
@@
 F 0 "R2" V 6000 4950 50  0000 C CNN
 F 1 "4k7" V 6100 4950 50  0000 C CNN
-F 2 "" V 6030 4950 30  0000 C CNN
+F 2 "Resistors_SMD:R_0805_HandSoldering" V 6030 4950 30  0001 C CNN
 F 3 "" H 6100 4950 30  0000 C CNN
 	1    6100 4950
@@
 F 0 "R5" V 6450 4800 50  0000 C CNN
 F 1 "4k7" V 6550 4800 50  0000 C CNN
-F 2 "" V 6480 4800 30  0000 C CNN
+F 2 "Resistors_SMD:R_0805_HandSoldering" V 6480 4800 30  0001 C CNN
 F 3 "" H 6550 4800 30  0000 C CNN
 	1    6550 4800
@@
 F 0 "P14" H 5650 3300 50  0000 C CNN
 F 1 "HUMID2" H 5850 3150 50  0000 C CNN
-F 2 "" H 5650 3100 60  0000 C CNN
+F 2 "autokiln:OSTOQ037151" H 5650 3100 60  0001 C CNN
 F 3 "" H 5650 3100 60  0000 C CNN
 	1    5650 3100
@@
 	5950 3200 5950 3300
 $Comp
-L GND #PWR50
+L GND #PWR053
 U 1 1 550D95EA
 P 5950 3300
-F 0 "#PWR50" H 5950 3050 60  0001 C CNN
+F 0 "#PWR053" H 5950 3050 60  0001 C CNN
 F 1 "GND" H 5950 3150 60  0000 C CNN
 F 2 "" H 5950 3300 60  0000 C CNN
@@
 F 0 "R4" V 6280 3000 50  0000 C CNN
 F 1 "1k" V 6200 3000 50  0000 C CNN
-F 2 "" V 6130 3000 30  0000 C CNN
+F 2 "Resistors_SMD:R_0805_HandSoldering" V 6130 3000 30  0001 C CNN
 F 3 "" H 6200 3000 30  0000 C CNN
 	1    6200 3000
@@
 F 0 "J3" H 8750 2600 50  0000 C CNN
 F 1 "HUMID PWR" H 9050 2400 50  0000 C CNN
-F 2 "" H 8750 2400 60  0000 C CNN
+F 2 "Pin_Headers:Pin_Header_Straight_1x03" H 8750 2400 60  0001 C CNN
 F 3 "" H 8750 2400 60  0000 C CNN
 	1    8750 2400
@@
 	8400 2500 8400 2600
 $Comp
-L +5V #PWR51
+L +5V #PWR054
 U 1 1 550DCB5E
 P 8400 2200
-F 0 "#PWR51" H 8400 2050 60  0001 C CNN
+F 0 "#PWR054" H 8400 2050 60  0001 C CNN
 F 1 "+5V" H 8400 2340 60  0000 C CNN
 F 2 "" H 8400 2200 60  0000 C CNN
@@
 $EndComp
 $Comp
-L VCC #PWR52
+L VCC #PWR055
 U 1 1 550DCB7A
 P 8400 2600
-F 0 "#PWR52" H 8400 2450 60  0001 C CNN
+F 0 "#PWR055" H 8400 2450 60  0001 C CNN
 F 1 "VCC" H 8400 2750 60  0000 C CNN
 F 2 "" H 8400 2600 60  0000 C CNN
