File: hardware/System.sch (KiCad schematic (older format))
At the start: 24 parts, among them P1 DEBUG, U1 STM32F070CBT6, U2 24LC512, X1 32kHz

Commit message: Schematic Draft Complete
Parts:
- removed C? (x11): 1uF, symbol C
- removed U?: NHD-C0220BiZ-FSW-FBW-3VM, symbol NHD-C0220BiZ-FSW-FBW-3VM
- removed U?: NHD-C12864LZ-FSW-FBW-3V3, symbol NHD-C12864LZ-FSW-FBW-3V3
- added C1, C2, C3, C5, C8: 100nF, symbol C
- added C4: 4u7, symbol C
- added R1: 3, symbol R
- added RV1: 10K, symbol POT
- added U1: NHD-0420AZ-FL-YBW-33V3, symbol NHD-0420AZ-FL-YBW-33V3
- gave numbers to parts that had none: 5
- renumbered C1 to C6, C2 to C7, U1 to U2, U2 to U3
Connections:
- net labels added: +5V, ADC_A0, ADC_A1, ADC_DOUT, ADC_PDWN, ADC_SCLK, HUMID_DATA1, HUMID_DATA2, LCD_BKL_EN, LCD_BKL_NEG, LCD_DB4, LCD_DB5, LCD_DB6, LCD_DB7, LCD_E, LCD_RS, LCD_RW
- net labels removed: HUMID_DATA, LCD_A0, LCD_C86, LCD_CS, LCD_RD, LCD_RST, LCD_SCL, LCD_SI, LCD_WR
- wire segments 151 -> 117
- no-connect marks 8 -> 6
Other:
- note added: "20x4 Character LCD"
- note added: "Backlight Current Limit:\n5V - 1.2V (V_CE_SAT) = 3.8V\n3.8V - 3.0V (V_BKL) = 0.8V\n0.8V = 300mA * 2.66 ohm"
- note added: "Backlight\n300mA, 3.0V"
- note added: "thruhole"
- note removed: "LCD \n20x2 CHARACTER"
- note removed: "LCD\n128x6\nPIXEL"
- note removed: "What to do with A/K?"
- note removed: "addr = 0x78"
- moved on the sheet: U3

Commit message: PCB mostly routed
Parts:
- added P16: UEXT, Pin_Headers:Pin_Header_Straight_2x05, symbol CONN_02X05
- C1, C2, C3, C4, C5, C6, C7, C8: footprint (none) -> Resistors_SMD:R_0805_HandSoldering
- P1: footprint (none) -> Pin_Headers:Pin_Header_Straight_1x04
- P2: footprint (none) -> Pin_Headers:Pin_Header_Straight_1x06
- R1: footprint (none) -> Resistors_ThroughHole:Resistor_Horizontal_RM10mm
- RV1: footprint (none) -> autokiln:BOURNS_TRIMMER_3303W
- SW1, SW2, SW3: footprint (none) -> autokiln:CK_Button_D6R
- SW4: value 318-ENC130175F-12PS -> PEC16-4215F-S0024; footprint (none) -> autokiln:BOURNS_Encoder_PEC16
- U1: footprint (none) -> autokiln:NHD-0420AZ-FL-GBW-33V3
- U2: footprint (none) -> Housings_QFP:LQFP-48_7x7mm_Pitch0.5mm
- U3: footprint (none) -> Housings_SOIC:SOIC-8_3.9x4.9mm_Pitch1.27mm
- X1: footprint (none) -> autokiln:Abracon_32KHz
Connections:
- net labels removed: ENC_C
- wire segments 117 -> 126
- no-connect marks 6 -> 11
Other:
- note added: "UEXT"
- moved on the sheet: P1, P2
