File: hardware/autokiln.kicad_pcb (KiCad board)
At the start: 2 copper layers, 185.4 x 130.8 mm, 71 parts, among them J1 GAIN JUMPER, J2 SPEED JUMPER, J3 HUMID PWR, K1 12V 250VAC 10A, K2 12V 250VAC 10A, K3 12V 250VAC 10A, K4 12V 250VAC 10A, K5 12V 250VAC 10A, P1 DEBUG, P10 VACUUM, P11 CONDITIONER, P12 BAROM, P13 HUMID1, P14 HUMID2, P15 VIN, P16 UEXT, P2 SWD, P3 LOAD CELL 1, P4 LOAD CELL 2, P5 LOAD CELL 3, P6 LOAD CELL 4, P7 HEATER, P8 DEHUMIDIFIER, P9 FAN, SW1 MENU, SW2 RESET, SW3 MANUAL, SW4 PEC16-4215F-S0024, SW5 PWR SWITCH, U1 NHD-0420AZ-FL-YBW-33V3, U2 STM32F070CBT6, U3 24LC512, U4 ADS1234, U5 ULQ2003, U6 L7805, U7 L4931, U8 KA278R12C, X1 32kHz

Commit message: PCB updates [wip]
Parts:
- moved C8 24.7 mm to (168.3, 45.2)
- moved C5 21.2 mm to (128.8, 58.5), turned to 0 degrees
- moved RV1 19.1 mm to (94.4, 27.9)
- moved C3 16.4 mm to (144.4, 81.9)
- moved C4 15.7 mm to (125.3, 75.2)
- moved C1 13.4 mm to (144.8, 50.9)
- moved C2 11.7 mm to (149.5, 63.2), turned to 270 degrees
- moved R2 11.1 mm to (168.0, 98.2)
- moved R5 9.03 mm to (168.0, 95.1)
- moved X1 8.93 mm to (116.8, 65.2)
- moved C7 6.08 mm to (121.0, 70.0), turned to 180 degrees
- moved C6 5.46 mm to (121.7, 59.8), turned to 180 degrees
- moved U2 3.38 mm to (139.4, 69.2)
- moved U3 2.62 mm to (138.7, 50.9)
- moved U5 2.61 mm to (163.2, 66.8)
Routing:
- net +5V: track 286.5 -> 426.5 mm, vias 1 -> 3
- net /System/SWDIO: track 5.27 -> 142.1 mm, vias 1 -> 4
- net ADC_A1: track 1.85 -> 124.2 mm, vias 1 -> 4
- net ADC_A0: track 4.82 -> 124.0 mm, vias 1 -> 4
- net /System/MANUAL: track 2.18 -> 114.9 mm, vias 1 -> 2
- net ADC_PDWN: track 4.48 -> 96.8 mm, vias 1 -> 4
- net /System/MENU: track 0.00 -> 90.9 mm, vias 0 -> 2
- net ADC_SCLK: track 6.24 -> 95.6 mm, vias 1 -> 4
- net VCC: track 339.9 -> 250.8 mm, vias 9 -> 5
- net ADC_DOUT: track 6.99 -> 94.7 mm, vias 1 -> 4
- net /System/RESET: track 2.41 -> 85.0 mm, vias 1 -> 2
- net /System/NRST: track 1.42 -> 83.3 mm, vias 1 -> 3
- net /System/ENC_A: track 3.48 -> 52.4 mm
- net /System/ENC_B: track 3.93 -> 51.0 mm
- net LCD_BKL_EN: track 0.82 -> 47.9 mm, vias 1 -> 4
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Other:
- board text added: "MANUAL"
- board text added: "MENU"
- board text added: "RESET"
