File: hardware/Relays.sch (KiCad schematic (older format))
At the start: 16 parts, among them K1 12V 250VAC 10A, K2 12V 250VAC 10A, K3 12V 250VAC 10A, K4 12V 250VAC 10A, K5 12V 250VAC 10A, P2 HEATER, P3 DEHUMIDIFIER, P4 FAN, P5 VACUUM, P6 CONDITIONER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

Commit message: Schematic Draft Complete
Parts:
- renumbered P5 to P10, P6 to P11, P2 to P7, P3 to P8, P4 to P9, U3 to U5
Connections:
- net LCD_BKL_NEG: now reaches U5.11 (OUT6)
- net LCD_BKL_EN: now reaches U5.6 (IN6)
- no-connect marks 9 -> 7
Changed lines of the file:
@@
 LIBS:valves
 LIBS:custom
+LIBS:autokiln-cache
 EELAYER 25 0
 EELAYER END
@@
 $EndComp
 $Comp
-L CONN_01X02 P2
+L CONN_01X02 P7
 U 1 1 5505EFEF
 P 10350 1450
-F 0 "P2" H 10350 1600 50  0000 C CNN
+F 0 "P7" H 10350 1600 50  0000 C CNN
 F 1 "HEATER" H 10350 1300 50  0000 C CNN
 F 2 "" H 10350 1450 60  0000 C CNN
@@
 $EndComp
 $Comp
-L CONN_01X02 P3
+L CONN_01X02 P8
 U 1 1 5505F07F
 P 10400 2400
-F 0 "P3" H 10400 2550 50  0000 C CNN
+F 0 "P8" H 10400 2550 50  0000 C CNN
 F 1 "DEHUMIDIFIER" H 10400 2250 50  0000 C CNN
 F 2 "" H 10400 2400 60  0000 C CNN
@@
 $EndComp
 $Comp
-L CONN_01X02 P4
+L CONN_01X02 P9
 U 1 1 5505F0F2
 P 10400 3350
-F 0 "P4" H 10400 3500 50  0000 C CNN
+F 0 "P9" H 10400 3500 50  0000 C CNN
 F 1 "FAN" H 10400 3200 50  0000 C CNN
 F 2 "" H 10400 3350 60  0000 C CNN
@@
 $EndComp
 $Comp
-L CONN_01X02 P5
+L CONN_01X02 P10
 U 1 1 5505F180
 P 10400 4300
-F 0 "P5" H 10400 4450 50  0000 C CNN
+F 0 "P10" H 10400 4450 50  0000 C CNN
 F 1 "VACUUM" H 10400 4150 50  0000 C CNN
 F 2 "" H 10400 4300 60  0000 C CNN
@@
 $EndComp
 $Comp
-L CONN_01X02 P6
+L CONN_01X02 P11
 U 1 1 5505F2A2
 P 10450 5250
-F 0 "P6" H 10450 5400 50  0000 C CNN
+F 0 "P11" H 10450 5400 50  0000 C CNN
 F 1 "CONDITIONER" H 10450 5100 50  0000 C CNN
 F 2 "" H 10450 5250 60  0000 C CNN
@@
 $EndComp
 $Comp
-L +12V #PWR07
+L +12V #PWR44
 U 1 1 550604B0
 P 6450 1800
-F 0 "#PWR07" H 6450 1650 60  0001 C CNN
+F 0 "#PWR44" H 6450 1650 60  0001 C CNN
 F 1 "+12V" H 6450 1940 60  0000 C CNN
 F 2 "" H 6450 1800 60  0000 C CNN
@@
 $EndComp
 $Comp
-L +12V #PWR08
+L +12V #PWR46
 U 1 1 55061014
 P 8800 1150
-F 0 "#PWR08" H 8800 1000 60  0001 C CNN
+F 0 "#PWR46" H 8800 1000 60  0001 C CNN
 F 1 "+12V" H 8800 1290 60  0000 C CNN
 F 2 "" H 8800 1150 60  0000 C CNN
@@
 	6450 2400 7200 2400
 Wire Wire Line
-	8800 1150 8800 1650
-Wire Wire Line
-	8800 1650 8800 2600
-Wire Wire Line
-	8800 2600 8800 3550
-Wire Wire Line
-	8800 3550 8800 4500
-Wire Wire Line
-	8800 4500 8800 5450
+	8800 1150 8800 5450
 Wire Wire Line
 	8800 1650 8900 1650
@@
 Text Label 7200 2400 2    60   ~ 0
 DEHUM_COIL
-$Comp
-L ULQ2003 U3
-U 1 1 55062CD9
-P 2750 4350
-F 0 "U3" H 2100 6300 60  0000 C CNN
-F 1 "ULQ2003" H 2200 6200 60  0000 C CNN
-F 2 "" H 2750 3650 60  0000 C CNN
-F 3 "" H 2750 3650 60  0000 C CNN
-	1    2750 4350
-	1    0    0    -1
-$EndComp
 Wire Wire Line
 	2950 3400 2850 3400
@@
 	2950 2400 2950 3400
 $Comp
-L +12V #PWR09
+L +12V #PWR40
 U 1 1 55062EC6
 P 2950 2400
-F 0 "#PWR09" H 2950 2250 60  0001 C CNN
+F 0 "#PWR40" H 2950 2250 60  0001 C CNN
 F 1 "+12V" H 2950 2540 60  0000 C CNN
 F 2 "" H 2950 2400 60  0000 C CNN
@@
 Wire Wire Line
 	1700 3100 850  3100
-NoConn ~ 1700 3200
 NoConn ~ 1700 3300
-NoConn ~ 2850 3200
 NoConn ~ 2850 3300
 Wire Wire Line
@@
 	1650 3400 1650 3450
 $Comp
-L GND #PWR010
+L GND #PWR39
 U 1 1 55063B3D
 P 1650 3450
-F 0 "#PWR010" H 1650 3200 60  0001 C CNN
+F 0 "#PWR39" H 1650 3200 60  0001 C CNN
 F 1 "GND" H 1650 3300 60  0000 C CNN
 F 2 "" H 1650 3450 60  0000 C CNN
@@
 $EndComp
 $Comp
-L +12V #PWR011
+L +12V #PWR45
 U 1 1 55063F10
 P 6450 3150
-F 0 "#PWR011" H 6450 3000 60  0001 C CNN
+F 0 "#PWR45" H 6450 3000 60  0001 C CNN
 F 1 "+12V" H 6450 3290 60  0000 C CNN
 F 2 "" H 6450 3150 60  0000 C CNN
@@
 $EndComp
 $Comp
-L +12V #PWR012
+L +12V #PWR41
 U 1 1 55064089
 P 5300 1800
-F 0 "#PWR012" H 5300 1650 60  0001 C CNN
+F 0 "#PWR41" H 5300 1650 60  0001 C CNN
 F 1 "+12V" H 5300 1940 60  0000 C CNN
 F 2 "" H 5300 1800 60  0000 C CNN
@@
 $EndComp
 $Comp
-L +12V #PWR013
+L +12V #PWR42
 U 1 1 550640A0
 P 5300 3150
-F 0 "#PWR013" H 5300 3000 60  0001 C CNN
+F 0 "#PWR42" H 5300 3000 60  0001 C CNN
 F 1 "+12V" H 5300 3290 60  0000 C CNN
 F 2 "" H 5300 3150 60  0000 C CNN
@@
 $EndComp
 $Comp
-L +12V #PWR014
+L +12V #PWR43
 U 1 1 55064173
 P 5300 4550
-F 0 "#PWR014" H 5300 4400 60  0001 C CNN
+F 0 "#PWR43" H 5300 4400 60  0001 C CNN
 F 1 "+12V" H 5300 4690 60  0000 C CNN
 F 2 "" H 5300 4550 60  0000 C CNN
@@
 Text GLabel 1800 1350 2    60   BiDi ~ 0
 STEAM
+Wire Wire Line
+	1700 3200 1450 3200
+$Comp
+L ULQ2003 U5
+U 1 1 55062CD9
+P 2750 4350
+F 0 "U5" H 2100 6300 60  0000 C CNN
+F 1 "ULQ2003" H 2200 6200 60  0000 C CNN
+F 2 "" H 2750 3650 60  0000 C CNN
+F 3 "" H 2750 3650 60  0000 C CNN
+	1    2750 4350
+	1    0    0    -1
+$EndComp
+Wire Wire Line
+	2850 3200 3050 3200
+Text GLabel 1450 3200 0    60   Input ~ 0
+LCD_BKL_EN
+Text GLabel 3050 3200 2    60   Output ~ 0
+LCD_BKL_NEG
 $EndSCHEMATC

Commit message: PCB mostly routed
Parts:
- D1, D2, D3, D4, D5: footprint (none) -> Diodes_ThroughHole:Diode_LED_5mm_round_vertical
- K1, K2, K3, K4, K5: footprint (none) -> Relays_ThroughHole:Relay_SANYOU_SRD_Series_Form_C
- P10, P11, P7, P8, P9: footprint (none) -> autokiln:OSTOQ020151
- U5: footprint (none) -> SMD_Packages:SO-16-N
Changed lines of the file:
@@
 encoding utf-8
 Sheet 4 6
-Title ""
-Date ""
-Rev ""
-Comp ""
+Title "Wood Drying Kiln Controller \"AutoKiln\""
+Date "Sat 21 Mar 2015"
+Rev "A1"
+Comp "Chris Merck"
 Comment1 ""
 Comment2 ""
@@
 F 0 "K1" H 9300 1550 50  0000 C CNN
 F 1 "12V 250VAC 10A" H 9450 900 50  0000 C CNN
-F 2 "" H 9300 1400 60  0000 C CNN
+F 2 "Relays_ThroughHole:Relay_SANYOU_SRD_Series_Form_C" H 9300 1400 60  0001 C CNN
 F 3 "" H 9300 1400 60  0000 C CNN
 	1    9300 1400
@@
 F 0 "K2" H 9300 2500 50  0000 C CNN
 F 1 "12V 250VAC 10A" H 9450 1850 50  0000 C CNN
-F 2 "" H 9300 2350 60  0000 C CNN
+F 2 "Relays_ThroughHole:Relay_SANYOU_SRD_Series_Form_C" H 9300 2350 60  0001 C CNN
 F 3 "" H 9300 2350 60  0000 C CNN
 	1    9300 2350
@@
 F 0 "K3" H 9300 3450 50  0000 C CNN
 F 1 "12V 250VAC 10A" H 9450 2800 50  0000 C CNN
-F 2 "" H 9300 3300 60  0000 C CNN
+F 2 "Relays_ThroughHole:Relay_SANYOU_SRD_Series_Form_C" H 9300 3300 60  0001 C CNN
 F 3 "" H 9300 3300 60  0000 C CNN
 	1    9300 3300
@@
 F 0 "K4" H 9300 4400 50  0000 C CNN
 F 1 "12V 250VAC 10A" H 9450 3750 50  0000 C CNN
-F 2 "" H 9300 4250 60  0000 C CNN
+F 2 "Relays_ThroughHole:Relay_SANYOU_SRD_Series_Form_C" H 9300 4250 60  0001 C CNN
 F 3 "" H 9300 4250 60  0000 C CNN
 	1    9300 4250
@@
 F 0 "K5" H 9300 5350 50  0000 C CNN
 F 1 "12V 250VAC 10A" H 9450 4700 50  0000 C CNN
-F 2 "" H 9300 5200 60  0000 C CNN
+F 2 "Relays_ThroughHole:Relay_SANYOU_SRD_Series_Form_C" H 9300 5200 60  0001 C CNN
 F 3 "" H 9300 5200 60  0000 C CNN
 	1    9300 5200
@@
 F 0 "P7" H 10350 1600 50  0000 C CNN
 F 1 "HEATER" H 10350 1300 50  0000 C CNN
-F 2 "" H 10350 1450 60  0000 C CNN
+F 2 "autokiln:OSTOQ020151" H 10350 1450 60  0001 C CNN
 F 3 "" H 10350 1450 60  0000 C CNN
 	1    10350 1450
@@
 F 0 "P8" H 10400 2550 50  0000 C CNN
 F 1 "DEHUMIDIFIER" H 10400 2250 50  0000 C CNN
-F 2 "" H 10400 2400 60  0000 C CNN
+F 2 "autokiln:OSTOQ020151" H 10400 2400 60  0001 C CNN
 F 3 "" H 10400 2400 60  0000 C CNN
 	1    10400 2400
@@
 F 0 "P9" H 10400 3500 50  0000 C CNN
 F 1 "FAN" H 10400 3200 50  0000 C CNN
-F 2 "" H 10400 3350 60  0000 C CNN
+F 2 "autokiln:OSTOQ020151" H 10400 3350 60  0001 C CNN
 F 3 "" H 10400 3350 60  0000 C CNN
 	1    10400 3350
@@
 F 0 "P10" H 10400 4450 50  0000 C CNN
 F 1 "VACUUM" H 10400 4150 50  0000 C CNN
-F 2 "" H 10400 4300 60  0000 C CNN
+F 2 "autokiln:OSTOQ020151" H 10400 4300 60  0001 C CNN
 F 3 "" H 10400 4300 60  0000 C CNN
 	1    10400 4300
@@
 F 0 "P11" H 10450 5400 50  0000 C CNN
 F 1 "CONDITIONER" H 10450 5100 50  0000 C CNN
-F 2 "" H 10450 5250 60  0000 C CNN
+F 2 "autokiln:OSTOQ020151" H 10450 5250 60  0001 C CNN
 F 3 "" H 10450 5250 60  0000 C CNN
 	1    10450 5250
@@
 F 0 "D4" V 6350 2250 50  0000 C CNN
 F 1 "12V LED" V 6550 2350 50  0000 C CNN
-F 2 "" H 6450 2150 60  0000 C CNN
+F 2 "Diodes_ThroughHole:Diode_LED_5mm_round_vertical" H 6450 2150 60  0001 C CNN
 F 3 "" H 6450 2150 60  0000 C CNN
 	1    6450 2150
@@
 $EndComp
 $Comp
-L +12V #PWR44
+L +12V #PWR042
 U 1 1 550604B0
 P 6450 1800
-F 0 "#PWR44" H 6450 1650 60  0001 C CNN
+F 0 "#PWR042" H 6450 1650 60  0001 C CNN
 F 1 "+12V" H 6450 1940 60  0000 C CNN
 F 2 "" H 6450 1800 60  0000 C CNN
@@
 $EndComp
 $Comp
-L +12V #PWR46
+L +12V #PWR043
 U 1 1 55061014
 P 8800 1150
-F 0 "#PWR46" H 8800 1000 60  0001 C CNN
+F 0 "#PWR043" H 8800 1000 60  0001 C CNN
 F 1 "+12V" H 8800 1290 60  0000 C CNN
 F 2 "" H 8800 1150 60  0000 C CNN
@@
 	2950 2400 2950 3400
 $Comp
-L +12V #PWR40
+L +12V #PWR044
 U 1 1 55062EC6
 P 2950 2400
-F 0 "#PWR40" H 2950 2250 60  0001 C CNN
+F 0 "#PWR044" H 2950 2250 60  0001 C CNN
 F 1 "+12V" H 2950 2540 60  0000 C CNN
 F 2 "" H 2950 2400 60  0000 C CNN
@@
 	1650 3400 1650 3450
 $Comp
-L GND #PWR39
+L GND #PWR045
 U 1 1 55063B3D
 P 1650 3450
-F 0 "#PWR39" H 1650 3200 60  0001 C CNN
+F 0 "#PWR045" H 1650 3200 60  0001 C CNN
 F 1 "GND" H 1650 3300 60  0000 C CNN
 F 2 "" H 1650 3450 60  0000 C CNN
@@
 F 0 "D5" V 6350 3600 50  0000 C CNN
 F 1 "12V LED" V 6550 3700 50  0000 C CNN
-F 2 "" H 6450 3500 60  0000 C CNN
+F 2 "Diodes_ThroughHole:Diode_LED_5mm_round_vertical" H 6450 3500 60  0001 C CNN
 F 3 "" H 6450 3500 60  0000 C CNN
 	1    6450 3500
@@
 $EndComp
 $Comp
-L +12V #PWR45
+L +12V #PWR046
 U 1 1 55063F10
 P 6450 3150
-F 0 "#PWR45" H 6450 3000 60  0001 C CNN
+F 0 "#PWR046" H 6450 3000 60  0001 C CNN
 F 1 "+12V" H 6450 3290 60  0000 C CNN
 F 2 "" H 6450 3150 60  0000 C CNN
@@
 F 0 "D1" V 5200 2250 50  0000 C CNN
 F 1 "12V LED" V 5400 2350 50  0000 C CNN
-F 2 "" H 5300 2150 60  0000 C CNN
+F 2 "Diodes_ThroughHole:Diode_LED_5mm_round_vertical" H 5300 2150 60  0001 C CNN
 F 3 "" H 5300 2150 60  0000 C CNN
 	1    5300 2150
@@
 $EndComp
 $Comp
-L +12V #PWR41
+L +12V #PWR047
 U 1 1 55064089
 P 5300 1800
-F 0 "#PWR41" H 5300 1650 60  0001 C CNN
+F 0 "#PWR047" H 5300 1650 60  0001 C CNN
 F 1 "+12V" H 5300 1940 60  0000 C CNN
 F 2 "" H 5300 1800 60  0000 C CNN
@@
 F 0 "D2" V 5200 3600 50  0000 C CNN
 F 1 "12V LED" V 5400 3700 50  0000 C CNN
-F 2 "" H 5300 3500 60  0000 C CNN
+F 2 "Diodes_ThroughHole:Diode_LED_5mm_round_vertical" H 5300 3500 60  0001 C CNN
 F 3 "" H 5300 3500 60  0000 C CNN
 	1    5300 3500
@@
 $EndComp
 $Comp
-L +12V #PWR42
+L +12V #PWR048
 U 1 1 550640A0
 P 5300 3150
-F 0 "#PWR42" H 5300 3000 60  0001 C CNN
+F 0 "#PWR048" H 5300 3000 60  0001 C CNN
 F 1 "+12V" H 5300 3290 60  0000 C CNN
 F 2 "" H 5300 3150 60  0000 C CNN
@@
 F 0 "D3" V 5200 5000 50  0000 C CNN
 F 1 "12V LED" V 5400 5100 50  0000 C CNN
-F 2 "" H 5300 4900 60  0000 C CNN
+F 2 "Diodes_ThroughHole:Diode_LED_5mm_round_vertical" H 5300 4900 60  0001 C CNN
 F 3 "" H 5300 4900 60  0000 C CNN
 	1    5300 4900
@@
 $EndComp
 $Comp
-L +12V #PWR43
+L +12V #PWR049
 U 1 1 55064173
 P 5300 4550
-F 0 "#PWR43" H 5300 4400 60  0001 C CNN
+F 0 "#PWR049" H 5300 4400 60  0001 C CNN
 F 1 "+12V" H 5300 4690 60  0000 C CNN
 F 2 "" H 5300 4550 60  0000 C CNN
@@
 F 0 "U5" H 2100 6300 60  0000 C CNN
 F 1 "ULQ2003" H 2200 6200 60  0000 C CNN
-F 2 "" H 2750 3650 60  0000 C CNN
+F 2 "SMD_Packages:SO-16-N" H 2750 3650 60  0001 C CNN
 F 3 "" H 2750 3650 60  0000 C CNN
 	1    2750 4350

Commit message: Autokiln Hardware Rev A
Parts:
- K1, K2, K3, K4, K5: value 12V 250VAC 10A -> 12V 250VAC 16A
Changed lines of the file:
@@
 P 9300 1400
 F 0 "K1" H 9300 1550 50  0000 C CNN
-F 1 "12V 250VAC 10A" H 9450 900 50  0000 C CNN
+F 1 "12V 250VAC 16A" H 9450 900 50  0000 C CNN
 F 2 "Relays_ThroughHole:Relay_SANYOU_SRD_Series_Form_C" H 9300 1400 60  0001 C CNN
 F 3 "" H 9300 1400 60  0000 C CNN
@@
 P 9300 2350
 F 0 "K2" H 9300 2500 50  0000 C CNN
-F 1 "12V 250VAC 10A" H 9450 1850 50  0000 C CNN
+F 1 "12V 250VAC 16A" H 9450 1850 50  0000 C CNN
 F 2 "Relays_ThroughHole:Relay_SANYOU_SRD_Series_Form_C" H 9300 2350 60  0001 C CNN
 F 3 "" H 9300 2350 60  0000 C CNN
@@
 P 9300 3300
 F 0 "K3" H 9300 3450 50  0000 C CNN
-F 1 "12V 250VAC 10A" H 9450 2800 50  0000 C CNN
+F 1 "12V 250VAC 16A" H 9450 2800 50  0000 C CNN
 F 2 "Relays_ThroughHole:Relay_SANYOU_SRD_Series_Form_C" H 9300 3300 60  0001 C CNN
 F 3 "" H 9300 3300 60  0000 C CNN
@@
 P 9300 4250
 F 0 "K4" H 9300 4400 50  0000 C CNN
-F 1 "12V 250VAC 10A" H 9450 3750 50  0000 C CNN
+F 1 "12V 250VAC 16A" H 9450 3750 50  0000 C CNN
 F 2 "Relays_ThroughHole:Relay_SANYOU_SRD_Series_Form_C" H 9300 4250 60  0001 C CNN
 F 3 "" H 9300 4250 60  0000 C CNN
@@
 P 9300 5200
 F 0 "K5" H 9300 5350 50  0000 C CNN
-F 1 "12V 250VAC 10A" H 9450 4700 50  0000 C CNN
+F 1 "12V 250VAC 16A" H 9450 4700 50  0000 C CNN
 F 2 "Relays_ThroughHole:Relay_SANYOU_SRD_Series_Form_C" H 9300 5200 60  0001 C CNN
 F 3 "" H 9300 5200 60  0000 C CNN
